File: stm32h7-hdmi-board-sodimm-module-hw.kicad_pcb (KiCad board)
At the start: 6 copper layers, 67.6 x 27.8 mm, 87 parts, among them J1 PCB-Edge_SODIMM_144_SDR, U1 IS42S86400F-7TL, U10 24AA024_TDFN, U2 IS42S86400F-7TL, U3 IS42S86400F-7TL, U4 IS42S86400F-7TL, U5 IS42S86400F-7TL, U6 IS42S86400F-7TL, U7 IS42S86400F-7TL, U8 IS42S86400F-7TL

Commit message: [#100919] Routing power
Parts:
- moved C24 26.7 mm to (151.1, 84.6)
- moved C8 23.4 mm to (116.1, 85.2)
- moved C48 23.0 mm to (135.7, 85.5)
- moved C16 21.9 mm to (133.7, 85.3)
- moved C56 17.2 mm to (148.8, 85.5)
- moved C66 11.9 mm to (168.6, 84.2)
- moved C40 11.6 mm to (118.4, 85.3)
- moved C64 10.7 mm to (165.9, 83.9)
- moved C32 7.70 mm to (170.5, 84.6)
- moved C23 5.46 mm to (142.7, 106.6)
- moved C31 4.99 mm to (157.8, 105.8), turned to -90 degrees
- moved C30 4.43 mm to (157.8, 101.3)
- moved C22 4.35 mm to (142.7, 101.5)
- moved C6 3.45 mm to (111.0, 101.5), turned to -90 degrees
- moved C7 3.45 mm to (111.0, 104.9), turned to 90 degrees
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Routing:
- net GND: track 22.1 -> 166.3 mm, vias 5 -> 17
- net +3.3V: track 29.8 -> 166.3 mm, vias 7 -> 19
- net /BA1: track 123.3 -> 126.2 mm
- net /SDR/A11: track 124.3 -> 127.0 mm
- net /BA0: track 122.5 -> 123.1 mm
