File: stm32h7-hdmi-board-sodimm-module-hw.kicad_pcb (KiCad board)
At the start: 6 copper layers, 67.6 x 27.8 mm, 87 parts, among them J1 PCB-Edge_SODIMM_144_SDR, U1 IS42S86400F-7TL, U10 24AA024_TDFN, U2 IS42S86400F-7TL, U3 IS42S86400F-7TL, U4 IS42S86400F-7TL, U5 IS42S86400F-7TL, U6 IS42S86400F-7TL, U7 IS42S86400F-7TL, U8 IS42S86400F-7TL

Commit message: [#100919] Add test points
Parts:
- added TP2: TP_1mm_SMD, antmicro-footprints:TP_SMD_1mm, F.Cu at (173.1, 92.4)
- added TP3: TP_1mm_SMD, antmicro-footprints:TP_SMD_1mm, F.Cu at (173.2, 94.8)
- added TP4: TP_1mm_SMD, antmicro-footprints:TP_SMD_1mm, F.Cu at (171.4, 113.8)
- moved TP1 11.5 mm to (173.2, 113.8)
Connections:
- TP1 pad 1: GND -> /EEPROM/EEPROM.SCL
Routing:
- net /EEPROM/EEPROM.SDA: track 11.0 -> 12.4 mm
- net +3.3V: track 233.9 -> 235.0 mm, vias 37 -> 38
- net /EEPROM/EEPROM.SCL: track 11.4 -> 12.5 mm
- net GND: track 230.5 -> 231.5 mm, vias 40 -> 42
