File: sodimm.kicad_sch (KiCad schematic)
At the start: 12 parts, among them J1 PCB-Edge_SODIMM_144_SDR

Commit message: [#101653] Change labels on schematic
Other:
- note added: "R1-R8 according to 144 Pin PC133 SDRAM SODIMM Reference Design"
- note removed: "R1-R8 according to 144 Pin PC133 SDRAM SO-DIMM Reference Design"
Changed lines of the file:
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@@
 		(comment 1 "www.antmicro.com")
 	)
-	(text "R1-R8 according to 144 Pin PC133\nSDRAM SO-DIMM Reference Design"
+	(text "R1-R8 according to 144 Pin PC133\nSDRAM SODIMM Reference Design"
 		(exclude_from_sim no)
 		(at 194.818 250.952 0)
